File: 3458A A3 66533 2021 KS SMD p1.1.kicad_sch (KiCad schematic)
At the start: 57 parts, among them U1 SN74LVC8T245PW, U10 HFBR1521Z, U11 LMS8117ADT-3.3, U12 LMS8117AMP-1.8, U2 SN74LVC8T245PW, U210 5M1270ZT144C5N, U3 SN74LVC8T245PW, U4 SN74LVC8T245PW, U5 SN74LVC8T245PW, U6 SN74LVC8T245PW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

Commit message: Corrected revision history table Following issues are addressed: Fixes #1 Fixes #2 Fixes #3 Fixes #4 Fixes #5 Fixes #6 Fixes #7 Fixes #9 Fixes #10
Parts:
- JD1: value Conn_02x05 -> JTAG 3.3V
Connections:
- net CK10S: now also U210.69 (IO1_69); no longer U210.66 (IO1_66)
- net _ADD2: now also U210.77 (IO2_77); no longer U210.44 (IO1_44)
- net _MSRST_F: now also U210.52 (IO1_52); no longer U210.53 (IO1_53)
- net _XINTR: now also U210.80 (IO2_80); no longer U210.28 (IO1_28)
Other:
- note removed: "3.3V JTAG"
- note removed: "Hard to tell if correct pin"
- moved on the sheet: C19, C20, C21, C22, C25, C26, C27, C28, C29, C3, C30, C34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
