File: 3458A A3 66533 2021 KS SMD p1.kicad_sch (KiCad schematic)
At the start: 177 parts, among them J2 Conn_01x02, P1 Conn_01x20, P2 Conn_01x20, Q401 MMBT3906, Q402 MMBT3906, Q403 PF5301, U131 74F112D, U213 74LCX00, U220 AT89LS51, U230 20MHz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

Commit message: Corrected revision history table Following issues are addressed: Fixes #1 Fixes #2 Fixes #3 Fixes #4 Fixes #5 Fixes #6 Fixes #7 Fixes #9 Fixes #10
Parts:
- C409-A1: value 250p? -> 470p
- C409-B1: value 260p? -> 10p
- CR241: value BAW56? -> MMBD1501; Comment Marking JC fits with BAW56, but diode reversed -> (none); Mfr. (none) -> onsemi; Mfr. Part Number BAW56? -> MMBD1501
Connections:
- net +3V3: now also JD2.2 (Pin_2)
- net A: now also JD2.6 (Pin_6)
- no-connect marks 29 -> 28
Other:
- note added: "66523: 1x510p"
- note added: "∑480p"
- note removed: "47R? (Marking unclear)"
- note removed: "Diode reversed in RoHS SMD revisions? (old schematic fits to old PCBs!) Marking JC fits with BAW56, but diode reversed No match for single diode with 1=A & 3=K"
- note removed: "Open? Should be GND"
- note removed: "wekomm: 1x510p"
- note removed: "∑510p?"
- moved on the sheet: C301, C302, C303, C351, C353, C400, C403, C404, C405, C4050, C4055, C4056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
