File: 3458A A3 66533 2021 KS SMD p2.kicad_sch (KiCad schematic)
At the start: 165 parts, among them J1 Conn_01x06, Q1 MMBF4393, Q11 MMBF4393, Q110 MMBF4392, Q12 MMBF4393, Q151 MMBT3904, Q2 MMBF4393, U110 LT1001, U111 AD817A, U112 AD848J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

Commit message: Corrected revision history table Following issues are addressed: Fixes #1 Fixes #2 Fixes #3 Fixes #4 Fixes #5 Fixes #6 Fixes #7 Fixes #9 Fixes #10
Parts:
- C119-A1: value 150p? -> 150p
- C119-B1: value 180p? -> 180p
- U180: Mfr. HP -> Keysight
Connections:
- no-connect marks 15 -> 16
Other:
- note added: "∑330p"
- note removed: "Have marking "JE" (BAV99?)"
- note removed: "No marking wekomm & KS"
- note removed: "wekomm: 1x330p"
- note removed: "∑330p?"
- moved on the sheet: C157, C158, C161, C162, C166, C167, Q151, R157, R158, R159, R161, R162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
